File: hardware/template/template.kicad_pcb (KiCad board)
At the start: 2 copper layers, 94 x 94 mm, 1 part, among them J1 Conn_02x20_Odd_Even

Commit message: Update template.kicad_pcb
Routing:
- net unconnected-(J1-Pin_8-Pad8): track 9.94 -> 0.00 mm, vias 1 -> 0
- net unconnected-(J1-Pin_40-Pad40): track 9.94 -> 0.00 mm, vias 1 -> 0
- net unconnected-(J1-Pin_4-Pad4): track 9.94 -> 0.00 mm, vias 1 -> 0
- net unconnected-(J1-Pin_38-Pad38): track 9.94 -> 0.00 mm, vias 1 -> 0
- net unconnected-(J1-Pin_36-Pad36): track 9.94 -> 0.00 mm, vias 1 -> 0
- net unconnected-(J1-Pin_32-Pad32): track 9.94 -> 0.00 mm, vias 1 -> 0
- net unconnected-(J1-Pin_30-Pad30): track 9.94 -> 0.00 mm, vias 1 -> 0
- net unconnected-(J1-Pin_24-Pad24): track 9.94 -> 0.00 mm, vias 1 -> 0
- net unconnected-(J1-Pin_22-Pad22): track 9.94 -> 0.00 mm, vias 1 -> 0
- net unconnected-(J1-Pin_2-Pad2): track 9.94 -> 0.00 mm, vias 1 -> 0
- net unconnected-(J1-Pin_18-Pad18): track 9.94 -> 0.00 mm, vias 1 -> 0
- net unconnected-(J1-Pin_16-Pad16): track 9.94 -> 0.00 mm, vias 1 -> 0
- net unconnected-(J1-Pin_10-Pad10): track 9.94 -> 0.00 mm, vias 1 -> 0
- net unconnected-(J1-Pin_6-Pad6): track 9.94 -> 0.00 mm, vias 1 -> 0
- net unconnected-(J1-Pin_34-Pad34): track 9.94 -> 0.00 mm, vias 1 -> 0
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