File: hardware/transmitter/transmitter.kicad_sch (KiCad schematic)
At the start: 0 parts

Commit message: another one structure improvements
Parts:
- added J1: Conn_02x20_Odd_Even, Connector_PinHeader_2.54mm:PinHeader_2x20_P2.54mm_Horizontal, symbol Connector_Generic:Conn_02x20_Odd_Even
- added J10, J11, J12, J13, J14, J15, J16, J17, J18, J19, J2, J20, J21, J26, J27, J28, J29, J3, J30, J31, J32, J33, J34, J35, J36, J37, J38, J39, J4, J40, J41, J42, J43, J44, J45, J5, J6, J7, J8, J9: Conn_01x01, symbol Connector_Generic:Conn_01x01
Connections:
- new net: J1.6 (Pin_6), J28.1 (Pin_1)
- new net: J1.25 (Pin_25), J14.1 (Pin_1)
- new net: J1.20 (Pin_20), J35.1 (Pin_1)
- new net: J1.11 (Pin_11), J7.1 (Pin_1)
- new net: J1.7 (Pin_7), J5.1 (Pin_1)
- new net: J1.22 (Pin_22), J36.1 (Pin_1)
- new net: J1.34 (Pin_34), J42.1 (Pin_1)
- new net: J1.23 (Pin_23), J13.1 (Pin_1)
- new net: J1.19 (Pin_19), J11.1 (Pin_1)
- new net: J1.1 (Pin_1), J2.1 (Pin_1)
- new net: J1.10 (Pin_10), J30.1 (Pin_1)
- new net: J1.29 (Pin_29), J16.1 (Pin_1)
- new net: J1.36 (Pin_36), J43.1 (Pin_1)
- new net: J1.15 (Pin_15), J9.1 (Pin_1)
- new net: J1.21 (Pin_21), J12.1 (Pin_1)
- new net: J1.38 (Pin_38), J44.1 (Pin_1)
- new net: J1.2 (Pin_2), J26.1 (Pin_1)
- new net: J1.4 (Pin_4), J27.1 (Pin_1)
- new net: J1.12 (Pin_12), J31.1 (Pin_1)
- new net: J1.13 (Pin_13), J8.1 (Pin_1)
- new net: J1.14 (Pin_14), J32.1 (Pin_1)
- new net: J1.16 (Pin_16), J33.1 (Pin_1)
- new net: J1.17 (Pin_17), J10.1 (Pin_1)
- new net: J1.18 (Pin_18), J34.1 (Pin_1)
- new net: J1.24 (Pin_24), J37.1 (Pin_1)
- new net: J1.26 (Pin_26), J38.1 (Pin_1)
- new net: J1.27 (Pin_27), J15.1 (Pin_1)
- new net: J1.28 (Pin_28), J39.1 (Pin_1)
- new net: J1.3 (Pin_3), J3.1 (Pin_1)
- new net: J1.30 (Pin_30), J40.1 (Pin_1)
- new net: J1.31 (Pin_31), J17.1 (Pin_1)
- new net: J1.32 (Pin_32), J41.1 (Pin_1)
- new net: J1.33 (Pin_33), J18.1 (Pin_1)
- new net: J1.35 (Pin_35), J19.1 (Pin_1)
- new net: J1.37 (Pin_37), J20.1 (Pin_1)
- new net: J1.39 (Pin_39), J21.1 (Pin_1)
- new net: J1.40 (Pin_40), J45.1 (Pin_1)
- new net: J1.5 (Pin_5), J4.1 (Pin_1)
- new net: J1.8 (Pin_8), J29.1 (Pin_1)
- new net: J1.9 (Pin_9), J6.1 (Pin_1)
