File: hardware/3axis-magnitometer/3axis-magnitometer.kicad_pcb (KiCad board)
At the start: 2 copper layers, 94 x 94 mm, 85 parts, among them J1 Conn_01x08_Pin, J2 Micro_SD_Card, J3 AVR-JTAG-10, J4 AVR-ISP-6, Q1 BSS138, Q2 BSS138, U1 PCF8563T, U2 ATmega32A-A, U3 AMS1117-3.3, U4 AMS1117-3.3, U5 qmc5883l, Y1 32.768кГц, Y2 7.3728MHz

Commit message: Add files via upload
Parts:
- removed J1: Conn_01x08_Pin, Connector_PinHeader_2.54mm:PinHeader_2x04_P2.54mm_Vertical
- removed the J2 at (136.7, 88.3)
- removed Q1, Q2: BSS138, Package_TO_SOT_SMD:SOT-23
- removed R20, R21, R24, R25: 2.2k, Resistor_SMD:R_0805_2012Metric
- removed R22, R23: 0, Resistor_SMD:R_0805_2012Metric
- removed TP1, TP10, TP11, TP2, TP3, TP4, TP7, TP8, TP9: TestPoint, TestPoint:TestPoint_Pad_D1.0mm
- removed TP5: SCL, TestPoint:TestPoint_Pad_D1.0mm
- removed TP6: SDA, TestPoint:TestPoint_Pad_D1.0mm
- added C13: 0.22, Capacitor_SMD:C_0805_2012Metric, F.Cu at (198.1, 83.8)
- added C14: 100p, Capacitor_SMD:C_0805_2012Metric, F.Cu at (195.6, 86.4)
- added C19: 4.7, Capacitor_SMD:C_0805_2012Metric, F.Cu at (195.6, 90.5)
- added C28: 0.22, Capacitor_SMD:C_0805_2012Metric, F.Cu at (188.0, 81.3)
- added C29: 0.22, Capacitor_SMD:C_0805_2012Metric, F.Cu at (186.1, 87.5)
- added C30: 0.22, Capacitor_SMD:C_0805_2012Metric, F.Cu at (200.7, 88.9)
- added C31: 0.22, Capacitor_SMD:C_0805_2012Metric, F.Cu at (237.8, 94.2)
- added C32: 0.22, Capacitor_SMD:C_0805_2012Metric, F.Cu at (199.4, 62.2)
- added C33: 0.22, Capacitor_SMD:C_0805_2012Metric, F.Cu at (194.3, 62.2)
- added R6: 2.2k, Resistor_SMD:R_0805_2012Metric, F.Cu at (259.0, 92.4)
- added R7: 2.2k, Resistor_SMD:R_0805_2012Metric, F.Cu at (259.0, 95.4)
- added U3: ATmega1284P-A, Package_QFP:TQFP-44_10x10mm_P0.8mm, F.Cu at (159.3, 87.6)
- added U7: 74LVC2T45DC, Package_SO:VSSOP-8_2.3x2mm_P0.5mm, F.Cu at (191.1, 83.8)
- added U8: 74LVC2T45DC, Package_SO:VSSOP-8_2.3x2mm_P0.5mm, F.Cu at (191.1, 88.7)
- added U9: LSM6DS3, Package_LGA:LGA-14_3x2.5mm_P0.5mm_LayoutBorder3x4y, F.Cu at (195.6, 57.1)
- U2: value ATmega32A-A -> W25Q128JVS; footprint Package_QFP:TQFP-44_10x10mm_P0.8mm -> Package_SO:SOIC-8_5.3x5.3mm_P1.27mm
- Y2: value 7.3728MHz -> 8MHz; footprint Crystal:Crystal_SMD_EuroQuartz_EQ161-2Pin_3.2x1.5mm -> Crystal:Crystal_SMD_EuroQuartz_MQ2-2Pin_7.0x5.0mm
- moved C21 59.9 mm to (264.8, 41.7)
- moved U5 59.9 mm to (255.2, 50.8)
- moved C15 59.9 mm to (264.8, 50.5)
- moved C16 59.9 mm to (262.8, 41.7)
- moved C17 59.9 mm to (262.8, 50.5)
- moved C22 59.9 mm to (249.6, 41.7)
- moved C23 59.9 mm to (249.6, 50.5)
- moved C24 59.9 mm to (247.5, 41.7)
- moved C25 59.9 mm to (247.5, 50.5)
- moved C26 59.9 mm to (245.5, 41.7)
- moved C27 59.9 mm to (245.5, 50.5)
- moved R13 59.9 mm to (266.9, 41.7)
- moved U6 59.9 mm to (255.0, 41.7)
- moved C18 59.9 mm to (260.8, 41.7)
- moved C20 59.9 mm to (260.8, 50.5)
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- renumbered C13 to C15, C14 to C16, C15 to C17, C16 to C18, C17 to C20, C18 to C21, C19 to C22, C20 to C23, C21 to C24, C22 to C25, C23 to C26, C24 to C27, C5 to C4, C4 to C5, J3 to J2, J4 to J3, R11 to R10, R12 to R11, R13 to R12, R14 to R13, R19 to R14, R26 to R15, R5 to R2, R6 to R3, R7 to R4, R8 to R5, R9 to R8, R10 to R9, U3 to U5, U4 to U6
Connections:
- C10 pad 2: Net-(J3-VREF) -> Net-(J2-VREF)
- C11 pad 2: Net-(J3-VREF) -> Net-(J2-VREF)
- C12 pad 1: Net-(U2-AVCC) -> Net-(U3-AVCC)
- C4 pad 2: Net-(J2-VDD) -> Net-(U2-VCC)
- C5 pad 2: Net-(J2-VDD) -> Net-(U2-VCC)
- C6 pad 1: Net-(U2-XTAL1) -> Net-(U3-XTAL1)
- C7 pad 1: Net-(U2-XTAL2) -> Net-(U3-XTAL2)
- C8 pad 2: Net-(U2-AREF) -> Net-(U3-AREF)
- C9 pad 2: Net-(J3-VREF) -> Net-(J2-VREF)
- FB1 pad 2: Net-(U2-AVCC) -> Net-(U3-AVCC)
- FB2 pad 2: Net-(U5-AVDD) -> Net-(U4-VDD)
- J2 pad 4: Net-(J3-VREF) -> Net-(J2-VREF)
- J3 pad 2: Net-(J3-VREF) -> Net-(J2-VREF)
- R1 pad 2: Net-(R1-Pad2) -> +3.3V
- R10 pad 1: Net-(U2-AVCC) -> Net-(U3-AVCC)
- R10 pad 2: Net-(U2-PA2) -> Net-(U3-PA2)
- R11 pad 1: Net-(U2-PA2) -> Net-(U3-PA2)
- R2 pad 2: Net-(J2-VDD) -> Net-(U2-VCC)
- R3 pad 2: Net-(J3-VREF) -> Net-(J2-VREF)
- R4 pad 1: Net-(J3-VREF) -> Net-(J2-VREF)
- R5 pad 1: Net-(J3-VREF) -> Net-(J2-VREF)
- R8 pad 1: Net-(J3-VREF) -> Net-(J2-VREF)
- R8 pad 2: Net-(U2-PA3) -> Net-(U3-PA3)
- R9 pad 1: Net-(U2-PA3) -> Net-(U3-PA3)
- U1 pad 2: GND -> Net-(U1-OSCO)
- U1 pad 3: /INT -> /clock/INT
- U2 pad 1: /MOSI  -> /SS
- U2 pad 3: /SCK -> Net-(U2-VCC)
- U2 pad 4: /mc/~{RESET} -> GND
- U2 pad 5: Net-(J3-VREF) -> /MOSI 
- U2 pad 6: GND -> /SCK
- U2 pad 7: Net-(U2-XTAL2) -> Net-(U2-VCC)
- U2 pad 8: Net-(U2-XTAL1) -> Net-(U2-VCC)
- Y1 pad 2: GND -> Net-(U1-OSCO)
- Y2 pad 1: Net-(U2-XTAL1) -> Net-(U3-XTAL1)
- Y2 pad 2: Net-(U2-XTAL2) -> Net-(U3-XTAL2)
Routing:
- net Net-(J2-VREF): track 0.00 -> 94.3 mm, vias 0 -> 2
- net Net-(J3-VREF): track 82.3 -> 0.00 mm, vias 1 -> 0
- net /SCK: track 91.6 -> 27.0 mm, vias 1 -> 0
- net /INT: track 62.6 -> 0.00 mm, vias 2 -> 1
- net /DRDY: track 67.6 -> 5.95 mm, vias 2 -> 1
- net /MISO: track 75.5 -> 26.7 mm, vias 1 -> 0
- net +5V: track 65.7 -> 23.1 mm, vias 1 -> 0
- net /CLK0: track 45.4 -> 3.90 mm, vias 2 -> 0
- net /MOSI : track 68.7 -> 27.3 mm
- net /level_translator/UART_TX: track 35.6 -> 0.00 mm, vias 2 -> 0
- net +3.3V: track 144.6 -> 109.4 mm, vias 4 -> 7
- net /level_translator/UART_RX: track 34.8 -> 0.00 mm, vias 2 -> 0
- net +3.3VA: track 87.9 -> 54.6 mm
- net /level_translator/TX: track 32.8 -> 4.66 mm, vias 1 -> 0
- net /level_translator/UART_TX0: track 0.00 -> 26.3 mm, vias 0 -> 2
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Other:
- outline, holes or cut-outs redrawn

Commit message: начата новая трассировка
Parts:
- removed the C25 at (247.5, 50.5)
- removed the C25 at (189.4, 47.9)
- removed the C26 at (189.4, 50.0)
- removed the C26 at (245.5, 41.7)
- removed the C27 at (200.2, 41.1)
- removed the C27 at (245.5, 50.5)
- removed the C28 at (188.0, 81.3)
- removed the C28 at (200.3, 49.1)
- removed the C29 at (200.3, 46.5)
- removed the C29 at (186.1, 87.5)
- removed the R15 at (189.3, 52.1)
- removed the R15 at (176.7, 88.6)
- removed R18, R27, R28: 2.2k, Resistor_SMD:R_0805_2012Metric
- removed the R2 at (175.1, 65.4)
- removed the R2 at (169.5, 54.2)
- removed the R3 at (159.1, 97.9)
- removed the R3 at (169.5, 48.1)
- removed the R4 at (169.5, 46.0)
- removed the R4 at (144.5, 86.6)
- removed the U5 at (195.6, 48.3)
- removed the U5 at (255.2, 50.8)
- added C25: C, Capacitor_SMD:C_0805_2012Metric, F.Cu at (149.5, 66.4)
- added C26: C, Capacitor_SMD:C_0805_2012Metric, F.Cu at (152.5, 66.4)
- added C27: C, Capacitor_SMD:C_0805_2012Metric, F.Cu at (155.5, 66.4)
- added C28: C, Capacitor_SMD:C_0805_2012Metric, F.Cu at (158.6, 66.4)
- added C29: 0.22, Capacitor_SMD:C_0805_2012Metric, F.Cu at (194.7, 84.2)
- added C34: 0.22, Capacitor_SMD:C_0805_2012Metric, F.Cu at (209.7, 84.2)
- added C35: 0.22, Capacitor_SMD:C_0805_2012Metric, F.Cu at (180.5, 72.8)
- added C36: 0.22, Capacitor_SMD:C_0805_2012Metric, F.Cu at (183.5, 72.8)
- added J1: Conn_01x40_Pin, Connector_PinHeader_2.54mm:PinHeader_2x20_P2.54mm_Horizontal, F.Cu at (207.0, 124.5)
- added JP1: SolderJumper_2_Open, Jumper:SolderJumper-2_P1.3mm_Open_TrianglePad1.0x1.5mm, F.Cu at (195.0, 90.0)
- added JP2: SolderJumper_2_Open, Jumper:SolderJumper-2_P1.3mm_Open_TrianglePad1.0x1.5mm, F.Cu at (198.5, 90.0)
- added JP3: SolderJumper_2_Open, Jumper:SolderJumper-2_P1.3mm_Open_TrianglePad1.0x1.5mm, F.Cu at (202.1, 90.0)
- added JP4: SolderJumper_2_Open, Jumper:SolderJumper-2_P1.3mm_Open_TrianglePad1.0x1.5mm, F.Cu at (205.7, 90.0)
- added JP5: SolderJumper_3_Open, Jumper:SolderJumper-3_P2.0mm_Open_TrianglePad1.0x1.5mm_NumberLabels, F.Cu at (209.2, 90.0)
- added JP6: SolderJumper_3_Open, Jumper:SolderJumper-3_P2.0mm_Open_TrianglePad1.0x1.5mm_NumberLabels, F.Cu at (212.8, 90.0)
- added JP7: SolderJumper_3_Open, Jumper:SolderJumper-3_P2.0mm_Open_TrianglePad1.0x1.5mm_NumberLabels, F.Cu at (216.4, 90.0)
- added JP8: SolderJumper_3_Open, Jumper:SolderJumper-3_P2.0mm_Open_TrianglePad1.0x1.5mm_NumberLabels, F.Cu at (219.9, 90.0)
- added R15: 2.2k, Resistor_SMD:R_0805_2012Metric, F.Cu at (210.8, 79.8)
- added R2: 10, Resistor_SMD:R_0805_2012Metric, F.Cu at (176.4, 80.7)
- added R3: 10, Resistor_SMD:R_0805_2012Metric, F.Cu at (209.0, 107.6)
- added R4: 2.2k, Resistor_SMD:R_0805_2012Metric, F.Cu at (211.9, 107.6)
- added U10: SP3485CN, Package_SO:SOIC-8_3.9x4.9mm_P1.27mm, F.Cu at (203.1, 77.8)
- added U11: LSM6DS3, Package_LGA:LGA-14_3x2.5mm_P0.5mm_LayoutBorder3x4y, F.Cu at (181.0, 67.9)
- added U4: QMC5883P, Package_LGA:LGA-16_3x3mm_P0.5mm_LayoutBorder3x5y, F.Cu at (168.9, 64.8)
- added U5: AMS1117-3.3, Package_TO_SOT_SMD:SOT-223-3_TabPin2, F.Cu at (152.2, 82.4)
- C14: value 100p -> 0.22
- C15: value C -> 100p
- C19: value 4.7 -> C
- C2: value C_Polarized -> 22p; footprint Battery:Battery_Panasonic_CR2032-HFN_Horizontal_CircularHoles -> Capacitor_SMD:C_0805_2012Metric
- C24: value C -> 4.7
- C3: value 0.1 -> C_Polarized; footprint Capacitor_SMD:C_0805_2012Metric -> Battery:Battery_Panasonic_CR2032-HFN_Horizontal_CircularHoles
- C4: value 100p -> 0.1
- C5: value 0.22 -> 100p
- C6: value 22p -> 0.22
- C8: value 0.22 -> 22p
- R17: value 2.2k -> 10
- U9: value LSM6DS3 -> SP3485CN; footprint Package_LGA:LGA-14_3x2.5mm_P0.5mm_LayoutBorder3x4y -> Package_SO:SOIC-8_3.9x4.9mm_P1.27mm
- moved C21 118.9 mm to (149.5, 70.8), turned to 90 degrees
- moved C16 118.2 mm to (149.5, 75.3), turned to 90 degrees
- moved C17 113.0 mm to (152.5, 75.3), turned to 90 degrees
- moved C18 110.4 mm to (155.5, 75.3), turned to 90 degrees
- moved R12 108.2 mm to (161.5, 75.3)
- moved R13 107.8 mm to (164.5, 75.3)
- moved U6 102.9 mm to (160.5, 82.4), turned to 90 degrees
- moved C22 101.3 mm to (152.5, 70.8)
- moved C23 96.2 mm to (155.5, 70.8)
- moved C15 95.0 mm to (172.5, 72.8), turned to 90 degrees
- moved C24 93.6 mm to (158.6, 70.8)
- moved C20 88.1 mm to (175.5, 72.8), turned to 90 degrees
- moved J3 82.2 mm to (210.2, 114.7), turned to 90 degrees
- moved BT1 75.1 mm to (158.8, 119.9), turned to 90 degrees
- moved Y2 74.6 mm to (219.9, 104.8), turned to 90 degrees
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Connections:
- C12 pad 1: Net-(U3-AVCC) -> GND
- C12 pad 2: GND -> Net-(J2-VREF)
- C13 pad 1: Net-(U4-VDD) -> Net-(U3-AVCC)
- C15 pad 1: Net-(U5-VI) -> Net-(U4-VDD)
- C16 pad 1: Net-(U6-VI) -> Net-(U5-VI)
- C17 pad 1: Net-(U5-VI) -> Net-(U6-VI)
- C18 pad 1: Net-(U6-VI) -> Net-(U5-VI)
- C19 pad 1: Net-(U4-C1) -> Net-(U6-VI)
- C2 pad 1: Net-(BT1-+) -> Net-(U1-OSCO)
- C20 pad 1: Net-(U5-VI) -> Net-(U4-C1)
- C21 pad 1: Net-(U6-VI) -> Net-(U5-VI)
- C22 pad 1: +3.3VA -> Net-(U6-VI)
- C23 pad 1: +3.3V -> +3.3VA
- C24 pad 1: +3.3VA -> +3.3V
- C3 pad 1: GND -> Net-(BT1-+)
- C3 pad 2: Net-(BT1-+) -> GND
- C30 pad 1: Net-(U7-VCCB) -> Net-(U7-VCCA)
- C31 pad 1: Net-(U7-VCCB) -> Net-(U10-VCC)
- C32 pad 1: GND -> Net-(U10-VCC)
- C32 pad 2: +3.3VA -> GND
- C33 pad 1: GND -> Net-(U10-VCC)
- C33 pad 2: +3.3V -> GND
- C4 pad 2: Net-(U2-VCC) -> Net-(BT1-+)
- C6 pad 1: Net-(U3-XTAL1) -> GND
- C6 pad 2: GND -> Net-(U2-VCC)
- C7 pad 1: Net-(U3-XTAL2) -> Net-(U3-XTAL1)
- C8 pad 1: GND -> Net-(U3-XTAL2)
- C8 pad 2: Net-(U3-AREF) -> GND
- C9 pad 2: Net-(J2-VREF) -> Net-(U3-AREF)
- R16 pad 1: Net-(U5-DVDD) -> Net-(U10-VCC)
- R16 pad 2: /SDA -> Net-(U10-DE)
- R17 pad 1: Net-(U5-DVDD) -> Net-(U10-VCC)
- R17 pad 2: /SCL -> +3.3V
- U1 pad 3: /clock/INT -> unconnected-(U1-~{INT}-Pad3)
- U1 pad 7: /CLK0 -> unconnected-(U1-CLKO-Pad7)
- U3 pad 41: /CLK0 -> unconnected-(U3-PB1-Pad41)
- U7 pad 6: /level_translator/UART_TX1 -> Net-(JP3-B)
- U7 pad 7: /level_translator/UART_TX0 -> Net-(JP1-B)
- U7 pad 8: Net-(U7-VCCB) -> Net-(U10-VCC)
- U8 pad 6: /level_translator/UART_RX1 -> Net-(JP4-B)
- U8 pad 7: /level_translator/UART_RX0 -> Net-(JP2-B)
- U8 pad 8: Net-(U7-VCCB) -> Net-(U10-VCC)
- U9 pad 1: GND -> Net-(JP7-A)
- U9 pad 2: unconnected-(U9-SDX-Pad2) -> Net-(U9-DE)
- U9 pad 3: unconnected-(U9-SCX-Pad3) -> Net-(U9-DE)
- U9 pad 4: /imu/INT1 -> Net-(JP5-A)
- U9 pad 5: +3.3V -> GND
- U9 pad 6: GND -> /level_translator/485_1_A
- U9 pad 7: GND -> /level_translator/485_1_B
- U9 pad 8: +3.3VA -> Net-(U10-VCC)
Routing:
- net +3.3V: track 109.4 -> 0.00 mm, vias 7 -> 0
- net /SCL: track 100.9 -> 0.00 mm, vias 4 -> 0
- net /SDA: track 99.8 -> 0.00 mm, vias 4 -> 0
- net Net-(J2-VREF): track 94.3 -> 0.00 mm, vias 2 -> 0
- net +3.3VA: track 54.6 -> 0.00 mm, vias 3 -> 0
- net /mc/~{RESET}: track 49.9 -> 0.00 mm, vias 2 -> 0
- net Net-(BT1-+): track 36.0 -> 0.00 mm
- net GND: track 34.5 -> 0.00 mm, vias 34 -> 0
- net /MOSI : track 27.3 -> 0.00 mm, vias 1 -> 0
- net /SCK: track 27.0 -> 0.00 mm
- net /MISO: track 26.7 -> 0.00 mm
- net /level_translator/UART_TX0: track 26.3 -> 0.00 mm, vias 2 -> 0
- net Net-(U5-DVDD): track 25.6 -> 0.00 mm, vias 2 -> 0
- net /level_translator/UART_RX0: track 25.6 -> 0.00 mm, vias 2 -> 0
- net +5V: track 23.1 -> 0.00 mm
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
Commit message: трасировка магнитометра
Parts:
- added C37: 0.22, Capacitor_SMD:C_0805_2012Metric, F.Cu at (57.6, 56.9)
- added FB3: FerriteBead, Inductor_SMD:L_0805_2012Metric, F.Cu at (69.5, 60.7)
- added FB4: FerriteBead, Inductor_SMD:L_0805_2012Metric, F.Cu at (68.3, 56.9)
- JP1, JP2, JP3, JP4: footprint Jumper:SolderJumper-2_P1.3mm_Open_TrianglePad1.0x1.5mm -> Jumper:SolderJumper-2_P1.3mm_Open_Pad1.0x1.5mm
- JP5, JP6, JP7, JP8: footprint Jumper:SolderJumper-3_P2.0mm_Open_TrianglePad1.0x1.5mm_NumberLabels -> Jumper:SolderJumper-3_P1.3mm_Open_Pad1.0x1.5mm
- U2: footprint Package_SO:SOIC-8_5.3x5.3mm_P1.27mm -> Package_SO:SOIC-8_3.9x4.9mm_P1.27mm
- moved J3 176.5 mm to (38.5, 74.1)
- moved Y2 175.9 mm to (44.8, 87.7), turned to 180 degrees
- moved JP8 170.3 mm to (50.2, 103.7)
- moved R4 168.7 mm to (45.7, 78.6)
- moved JP6 167.8 mm to (45.6, 103.7)
- moved R16 167.5 mm to (47.9, 103.7), turned to -90 degrees
- moved C10 165.6 mm to (43.1, 78.6), turned to -90 degrees
- moved R5 164.3 mm to (55.1, 69.5), turned to 180 degrees
- moved C34 159.9 mm to (52.1, 111.2)
- moved U10 158.8 mm to (47.9, 111.2), turned to -90 degrees
- moved R17 158.6 mm to (61.2, 111.2)
- moved JP7 157.4 mm to (59.6, 103.7)
- moved C8 157.4 mm to (42.7, 92.1), turned to 0 degrees
- moved R11 155.8 mm to (61.1, 73.8), turned to 180 degrees
- moved R15 155.3 mm to (57.3, 103.7), turned to -90 degrees
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Connections:
- C35 pad 2: +3.3VA -> Net-(U11-VDD)
- C36 pad 2: +3.3V -> Net-(U11-CS)
- U11 pad 12: +3.3V -> Net-(U11-CS)
- U11 pad 5: +3.3V -> Net-(U11-CS)
- U11 pad 8: +3.3VA -> Net-(U11-VDD)
Routing:
- net +3.3VA: track 0.00 -> 147.5 mm, vias 0 -> 5
- net +3.3V: track 0.00 -> 138.4 mm, vias 0 -> 6
- net /SCL: track 0.00 -> 107.2 mm, vias 0 -> 4
- net /SDA: track 0.00 -> 103.8 mm, vias 0 -> 4
- net Net-(J2-VREF): track 0.00 -> 97.9 mm, vias 0 -> 6
- net Net-(U10-VCC): track 0.00 -> 96.8 mm, vias 0 -> 8
- net Net-(JP3-B): track 0.00 -> 62.0 mm, vias 0 -> 2
- net Net-(JP1-B): track 0.00 -> 55.7 mm, vias 0 -> 4
- net +5V: track 0.00 -> 53.4 mm, vias 0 -> 2
- net Net-(JP4-B): track 0.00 -> 47.4 mm, vias 0 -> 2
- net Net-(JP2-B): track 0.00 -> 42.3 mm, vias 0 -> 4
- net /MISO: track 0.00 -> 39.7 mm
- net GND: track 0.00 -> 39.6 mm, vias 0 -> 49
- net /mc/~{RESET}: track 0.00 -> 38.4 mm, vias 0 -> 1
- net /level_translator/TX1: track 0.00 -> 36.4 mm, vias 0 -> 2
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Other:
- outline, holes or cut-outs redrawn
