File: hardware/3axis-magnitometer/3axis-magnitometer.kicad_pcb (KiCad board)
At the start: 2 copper layers, 94 x 94 mm, 91 parts, among them J1 Conn_01x40_Pin, J2 AVR-JTAG-10, J3 AVR-ISP-6, U1 PCF8563T, U10 LSM6DS3, U2 W25Q128JVS, U3 ATmega1284P-A, U4 QMC5883P, U5 AMS1117-3.3, U6 AMS1117-3.3, U7 SP3485CN, U8 SP3485CN, U9 TXB0104PW, Y1 32.768кГц, Y2 8MHz

Commit message: исправления трассировки
Parts:
- moved R15 0.64 mm to (120.8, 94.1)
- moved R16 0.62 mm to (111.4, 94.1)
- moved C33 0.51 mm to (136.7, 98.7)
- moved C32 0.51 mm to (136.7, 103.3)
- moved C8 0.25 mm to (111.1, 81.9)
- moved U7 0.17 mm to (120.7, 100.9)
- moved C11 0.16 mm to (106.1, 68.5)
- moved C9 0.13 mm to (105.5, 81.9)
- moved R6 0.13 mm to (123.4, 58.4)
Routing:
- net /mc/TCK: track 19.3 -> 24.8 mm
- net /level_translator/TX0: track 28.4 -> 25.5 mm
- net Net-(U7-VCC): track 78.2 -> 75.3 mm
- net /mc/TDO: track 19.7 -> 22.5 mm
- net /level_translator/UART_RX0: track 30.5 -> 33.2 mm
- net /SDA: track 94.5 -> 97.0 mm, vias 4 -> 3
- net /SCL: track 98.4 -> 100.7 mm, vias 4 -> 2
- net /SS: track 15.5 -> 13.2 mm
- net Net-(J2-VREF): track 98.7 -> 100.5 mm
- net /mc/~{RESET}: track 38.5 -> 39.8 mm
- net +3.3V: track 136.6 -> 135.6 mm
- net /level_translator/TX1: track 31.3 -> 32.2 mm, vias 1 -> 0
- net /level_translator/UART_TX0: track 20.4 -> 21.3 mm
- net Net-(U7-DE): track 7.13 -> 6.18 mm
- net /mc/TMS: track 26.6 -> 27.5 mm
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
Commit message: релиз
Parts:
- added GLADOLUS-1: LOGO, IONISTOR:GLADIOLUS, F.Cu at (98.8, 109.5)
- added REF**: MountingHole_4.3mm_M4_ISO14580, MountingHole:MountingHole_4.3mm_M4_ISO14580, F.Cu at (98.9, 42.6)
- added REF**: MountingHole_4.3mm_M4_ISO14580, MountingHole:MountingHole_4.3mm_M4_ISO14580, F.Cu at (172.7, 42.7)
- added REF**: MountingHole_4.3mm_M4_ISO14580, MountingHole:MountingHole_4.3mm_M4_ISO14580, F.Cu at (95.8, 128.3)
- added REF**: MountingHole_4.3mm_M4_ISO14580, MountingHole:MountingHole_4.3mm_M4_ISO14580, F.Cu at (175.8, 128.3)
- moved REF** 65.9 mm to (161.2, 50.3)
- moved C1 0.98 mm to (159.3, 67.1)
- moved C17 0.98 mm to (155.8, 100.9)
- moved C19 0.98 mm to (157.9, 100.9)
- moved C2 0.98 mm to (159.3, 59.7)
- moved C20 0.98 mm to (172.9, 100.9)
- moved C21 0.98 mm to (147.6, 46.5)
- moved C23 0.98 mm to (175.2, 100.9)
- moved C25 0.98 mm to (154.3, 88.9)
- moved C26 0.98 mm to (171.7, 89.0)
- moved C27 0.98 mm to (156.9, 88.9)
- moved C28 0.98 mm to (174.3, 89.0)
- moved C3 0.98 mm to (169.4, 76.0)
- moved C32 0.98 mm to (135.8, 103.0)
- moved C33 0.98 mm to (135.8, 98.5)
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Routing:
- net GND: track 33.3 -> 49.5 mm
Other:
- outline, holes or cut-outs redrawn
- board text added: "Magnetometer"
- board text added: "Аccelerometer"
