File: hardware/3axis-magnitometer/magnitometr.kicad_sch (KiCad schematic)
At the start: 11 parts, among them U5 qmc5883l

Commit message: Add files via upload
Parts:
- removed C25, C26, C27, C29: 0.22, Capacitor_SMD:C_0805_2012Metric, symbol Device:C
- removed C28: 4.7, Capacitor_SMD:C_0805_2012Metric, symbol Device:C
- removed R15: 10, Resistor_SMD:R_0805_2012Metric, symbol Device:R
- removed R16, R17, R18: 2.2k, Resistor_SMD:R_0805_2012Metric, symbol Device:R
- removed U5: qmc5883l, Package_LGA:LGA-16_3x3mm_P0.5mm, symbol Sensor_Magnetic:qmc5883l
- added C13: 0.22, Capacitor_SMD:C_0805_2012Metric, symbol Device:C
- added C14: 100p, Capacitor_SMD:C_0805_2012Metric, symbol Device:C
- added C19: 4.7, Capacitor_SMD:C_0805_2012Metric, symbol Device:C
- added U4: QMC5883P, MODULE, symbol common:QMC5883P
Connections:
- net GND: now also C13.2, C14.2, C19.2, U4.11 (GND), U4.9 (GND)
- net SCL: now also U4.1 (SCL)
- net SDA: now also U4.16 (SDA)
- net at FB2.2: now also C13.1, C14.1, U4.2 (VDD)
- new net: C19.1, U4.10 (C1)
- no-connect marks 0 -> 5
Other:
- moved on the sheet: FB2

Commit message: начата новая трассировка
Parts:
- U4: footprint MODULE -> Package_LGA:LGA-16_3x3mm_P0.5mm_LayoutBorder3x5y
- renumbered C13 to C14, C14 to C15, C19 to C20
Changed lines of the file:
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@@
 		(on_board yes)
 		(dnp no)
-		(property "Reference" "C13"
+		(property "Reference" "C14"
 			(at 121.92 77.216 0)
 			(effects
@@
 			(project "3axis-magnitometer"
 				(path "/c590c88d-27c9-4e5a-a435-a42d9de70c1c/0bdc1534-3886-4ec0-96c3-23dabfd87e22"
-					(reference "C13")
+					(reference "C14")
 					(unit 1)
 				)
@@
 		(on_board yes)
 		(dnp no)
-		(property "Reference" "C14"
+		(property "Reference" "C15"
 			(at 132.08 77.216 0)
 			(effects
@@
 			(project "3axis-magnitometer"
 				(path "/c590c88d-27c9-4e5a-a435-a42d9de70c1c/0bdc1534-3886-4ec0-96c3-23dabfd87e22"
-					(reference "C14")
+					(reference "C15")
 					(unit 1)
 				)
@@
 			)
 		)
-		(property "Footprint" "MODULE"
+		(property "Footprint" "Package_LGA:LGA-16_3x3mm_P0.5mm_LayoutBorder3x5y"
 			(at 157.48 63.5 0)
 			(effects
@@
 		(dnp no)
 		(fields_autoplaced yes)
-		(property "Reference" "C19"
+		(property "Reference" "C20"
 			(at 165.1 85.0899 0)
 			(effects
@@
 			(project "3axis-magnitometer"
 				(path "/c590c88d-27c9-4e5a-a435-a42d9de70c1c/0bdc1534-3886-4ec0-96c3-23dabfd87e22"
-					(reference "C19")
-					(unit 1)
-				)
+					(reference "C20")
+					(unit 1)
+				)

Commit message: Финальные правки трассировки
Parts:
- renumbered C14 to C15, C15 to C16, C20 to C21
Changed lines of the file:
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@@
 		(on_board yes)
 		(dnp no)
-		(property "Reference" "C14"
+		(property "Reference" "C15"
 			(at 121.92 77.216 0)
 			(effects
@@
 			(project "3axis-magnitometer"
 				(path "/c590c88d-27c9-4e5a-a435-a42d9de70c1c/0bdc1534-3886-4ec0-96c3-23dabfd87e22"
-					(reference "C14")
+					(reference "C15")
 					(unit 1)
 				)
@@
 		(on_board yes)
 		(dnp no)
-		(property "Reference" "C15"
+		(property "Reference" "C16"
 			(at 132.08 77.216 0)
 			(effects
@@
 			(project "3axis-magnitometer"
 				(path "/c590c88d-27c9-4e5a-a435-a42d9de70c1c/0bdc1534-3886-4ec0-96c3-23dabfd87e22"
-					(reference "C15")
+					(reference "C16")
 					(unit 1)
 				)
@@
 		(dnp no)
 		(fields_autoplaced yes)
-		(property "Reference" "C20"
+		(property "Reference" "C21"
 			(at 165.1 85.0899 0)
 			(effects
@@
 			(project "3axis-magnitometer"
 				(path "/c590c88d-27c9-4e5a-a435-a42d9de70c1c/0bdc1534-3886-4ec0-96c3-23dabfd87e22"
-					(reference "C20")
-					(unit 1)
-				)
+					(reference "C21")
+					(unit 1)
+				)
