File: hardware/3axis-magnitometer/mc.kicad_sch (KiCad schematic)
At the start: 19 parts, among them J3 AVR-JTAG-10, J4 AVR-ISP-6, U2 ATmega32A-A, Y2 7.3728MHz

Commit message: Add files via upload
Parts:
- removed U2: ATmega32A-A, Package_QFP:TQFP-44_10x10mm_P0.8mm, symbol MCU_Microchip_ATmega:ATmega32A-A
- added R6, R7: 2.2k, Resistor_SMD:R_0805_2012Metric, symbol Device:R
- added U3: ATmega1284P-A, Package_QFP:TQFP-44_10x10mm_P0.8mm, symbol MCU_Microchip_ATmega:ATmega1284P-A
- Y2: value 7.3728MHz -> 8MHz; footprint Crystal:Crystal_SMD_EuroQuartz_EQ161-2Pin_3.2x1.5mm -> Crystal:Crystal_SMD_EuroQuartz_MQ2-2Pin_7.0x5.0mm
- renumbered J3 to J2, J4 to J3, R11 to R10, R12 to R11, R6 to R3, R7 to R4, R8 to R5, R9 to R8, R10 to R9
Connections:
- net CLK0: now also U3.41 (PB1)
- net DRDY: now also U3.36 (PA1)
- net GND: now also U3.18 (GND), U3.28 (GND), U3.39 (GND), U3.6 (GND)
- net MISO: now also U3.2 (PB6)
- net MOSI : now also U3.1 (PB5)
- net RX0: now also U3.9 (PD0)
- net SCK: now also U3.3 (PB7)
- net SCL: now also R6.2, U3.19 (PC0)
- net SDA: now also R7.2, U3.20 (PC1)
- net SS: now also U3.44 (PB4)
- net TCK: now also U3.21 (PC2)
- net TDI: now also U3.24 (PC5)
- net TDO: now also U3.23 (PC4)
- net TMS: now also U3.22 (PC3)
- net TX0: now also U3.10 (PD1)
- net ~{RESET}: now also U3.4 (~{RESET})
- net at C7.1, Y2.2: now also U3.7 (XTAL2)
- net at C6.1, Y2.1: now also U3.8 (XTAL1)
- net at C10.2, C11.2, C9.2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: now also R6.1, R7.1, U3.17 (VCC), U3.38 (VCC), U3.5 (VCC)
- net at R10.2, R11.1: now also U3.35 (PA2)
- net at C12.1, FB1.2, R10.1: now also U3.27 (AVCC)
- net at C8.2: now also U3.29 (AREF)
- net at R8.2, R9.1: now also U3.34 (PA3)
- new net RX1: U3.11 (PD2)
- new net TX1: U3.12 (PD3)
Other:
- moved on the sheet: C12, R4

Commit message: начата новая трассировка
Parts:
- renumbered C9 to C10, C10 to C11, C11 to C12, C12 to C13, C6 to C7, C7 to C8, C8 to C9
Connections:
- net CLK0: no longer names the net of U3.41 (PB1)
- no-connect marks 22 -> 23
Changed lines of the file:
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@@
+	)
+	(no_connect
+		(at 93.98 88.9)
 	)
 	(no_connect
@@
 	(wire
 		(pts
-			(xy 214.63 25.4) (xy 214.63 35.56)
+			(xy 214.63 27.94) (xy 214.63 35.56)
 		)
 		(stroke
@@
 	(wire
 		(pts
-			(xy 93.98 88.9) (xy 267.97 88.9)
-		)
-		(stroke
-			(width 0)
-			(type default)
-		)
-	)
-	(wire
-		(pts
 			(xy 170.18 71.12) (xy 170.18 149.86)
 		)
@@
 	(wire
 		(pts
-			(xy 243.84 35.56) (xy 243.84 25.4)
+			(xy 243.84 35.56) (xy 243.84 27.94)
 		)
 		(stroke
@@
 	(wire
 		(pts
-			(xy 243.84 25.4) (xy 214.63 25.4)
+			(xy 243.84 27.94) (xy 214.63 27.94)
 		)
 		(stroke
@@
 	(label "SCK"
 		(at 257.81 104.14 0)
-		(effects
-			(font
-				(size 1.27 1.27)
-			)
-			(justify left bottom)
-		)
-	)
-	(label "CLK0"
-		(at 257.81 88.9 0)
 		(effects
 			(font
@@
 		(shape input)
 		(at 267.97 132.08 0)
-		(effects
-			(font
-				(size 1.27 1.27)
-			)
-			(justify left)
-		)
-	)
-	(hierarchical_label "CLK0"
-		(shape input)
-		(at 267.97 88.9 0)
 		(effects
 			(font
@@
 		(on_board yes)
 		(dnp no)
-		(property "Reference" "C7"
+		(property "Reference" "C8"
 			(at 23.114 91.694 90)
 			(effects
@@
 			(project "3axis-magnitometer"
 				(path "/c590c88d-27c9-4e5a-a435-a42d9de70c1c/8b451e59-e543-47cc-9c8c-0cf4f90bdb2a"
-					(reference "C7")
+					(reference "C8")
 					(unit 1)
 				)
@@
 		(on_board yes)
 		(dnp no)
-		(property "Reference" "C11"
+		(property "Reference" "C12"
 			(at 263.144 27.178 0)
 			(effects
@@
 			(project "3axis-magnitometer"
 				(path "/c590c88d-27c9-4e5a-a435-a42d9de70c1c/8b451e59-e543-47cc-9c8c-0cf4f90bdb2a"
-					(reference "C11")
+					(reference "C12")
 					(unit 1)
 				)
@@
 		(on_board yes)
 		(dnp no)
-		(property "Reference" "C12"
+		(property "Reference" "C13"
 			(at 277.114 26.924 0)
 			(effects
@@
 			(project ""
 				(path "/c590c88d-27c9-4e5a-a435-a42d9de70c1c/8b451e59-e543-47cc-9c8c-0cf4f90bdb2a"
-					(reference "C12")
+					(reference "C13")
 					(unit 1)
 				)
@@
 		(on_board yes)
 		(dnp no)
-		(property "Reference" "C10"
+		(property "Reference" "C11"
 			(at 256.54 27.178 0)
 			(effects
@@
 			(project "3axis-magnitometer"
 				(path "/c590c88d-27c9-4e5a-a435-a42d9de70c1c/8b451e59-e543-47cc-9c8c-0cf4f90bdb2a"
-					(reference "C10")
+					(reference "C11")
 					(unit 1)
 				)
@@
 		(on_board yes)
 		(dnp no)
-		(property "Reference" "C9"
+		(property "Reference" "C10"
 			(at 250.19 27.178 0)
 			(effects
@@
 			(project "3axis-magnitometer"
 				(path "/c590c88d-27c9-4e5a-a435-a42d9de70c1c/8b451e59-e543-47cc-9c8c-0cf4f90bdb2a"
-					(reference "C9")
+					(reference "C10")
 					(unit 1)
 				)
@@
 		(on_board yes)
 		(dnp no)
-		(property "Reference" "C8"
+		(property "Reference" "C9"
 			(at 48.26 101.6 0)
 			(effects
@@
 			(project "3axis-magnitometer"
 				(path "/c590c88d-27c9-4e5a-a435-a42d9de70c1c/8b451e59-e543-47cc-9c8c-0cf4f90bdb2a"
-					(reference "C8")
+					(reference "C9")
 					(unit 1)
 				)
@@
 		(on_board yes)
 		(dnp no)
-		(property "Reference" "C6"
+		(property "Reference" "C7"
 			(at 12.954 89.154 90)
 			(effects
@@
 			(project "3axis-magnitometer"
 				(path "/c590c88d-27c9-4e5a-a435-a42d9de70c1c/8b451e59-e543-47cc-9c8c-0cf4f90bdb2a"
-					(reference "C6")
-					(unit 1)
-				)
+					(reference "C7")
+					(unit 1)
+				)

Commit message: Финальные правки трассировки
Parts:
- renumbered C9 to C10, C10 to C11, C11 to C12, C12 to C13, C13 to C14, C7 to C8, C8 to C9
Changed lines of the file:
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@@
 		(on_board yes)
 		(dnp no)
-		(property "Reference" "C8"
+		(property "Reference" "C9"
 			(at 23.114 91.694 90)
 			(effects
@@
 			(project "3axis-magnitometer"
 				(path "/c590c88d-27c9-4e5a-a435-a42d9de70c1c/8b451e59-e543-47cc-9c8c-0cf4f90bdb2a"
-					(reference "C8")
+					(reference "C9")
 					(unit 1)
 				)
@@
 		(on_board yes)
 		(dnp no)
-		(property "Reference" "C12"
+		(property "Reference" "C13"
 			(at 263.144 27.178 0)
 			(effects
@@
 			(project "3axis-magnitometer"
 				(path "/c590c88d-27c9-4e5a-a435-a42d9de70c1c/8b451e59-e543-47cc-9c8c-0cf4f90bdb2a"
-					(reference "C12")
+					(reference "C13")
 					(unit 1)
 				)
@@
 		(on_board yes)
 		(dnp no)
-		(property "Reference" "C13"
+		(property "Reference" "C14"
 			(at 277.114 26.924 0)
 			(effects
@@
 			(project ""
 				(path "/c590c88d-27c9-4e5a-a435-a42d9de70c1c/8b451e59-e543-47cc-9c8c-0cf4f90bdb2a"
-					(reference "C13")
+					(reference "C14")
 					(unit 1)
 				)
@@
 		(on_board yes)
 		(dnp no)
-		(property "Reference" "C11"
+		(property "Reference" "C12"
 			(at 256.54 27.178 0)
 			(effects
@@
 			(project "3axis-magnitometer"
 				(path "/c590c88d-27c9-4e5a-a435-a42d9de70c1c/8b451e59-e543-47cc-9c8c-0cf4f90bdb2a"
-					(reference "C11")
+					(reference "C12")
 					(unit 1)
 				)
@@
 		(on_board yes)
 		(dnp no)
-		(property "Reference" "C10"
+		(property "Reference" "C11"
 			(at 250.19 27.178 0)
 			(effects
@@
 			(project "3axis-magnitometer"
 				(path "/c590c88d-27c9-4e5a-a435-a42d9de70c1c/8b451e59-e543-47cc-9c8c-0cf4f90bdb2a"
-					(reference "C10")
+					(reference "C11")
 					(unit 1)
 				)
@@
 		(on_board yes)
 		(dnp no)
-		(property "Reference" "C9"
+		(property "Reference" "C10"
 			(at 48.26 101.6 0)
 			(effects
@@
 			(project "3axis-magnitometer"
 				(path "/c590c88d-27c9-4e5a-a435-a42d9de70c1c/8b451e59-e543-47cc-9c8c-0cf4f90bdb2a"
-					(reference "C9")
+					(reference "C10")
 					(unit 1)
 				)
@@
 		(on_board yes)
 		(dnp no)
-		(property "Reference" "C7"
+		(property "Reference" "C8"
 			(at 12.954 89.154 90)
 			(effects
@@
 			(project "3axis-magnitometer"
 				(path "/c590c88d-27c9-4e5a-a435-a42d9de70c1c/8b451e59-e543-47cc-9c8c-0cf4f90bdb2a"
-					(reference "C7")
-					(unit 1)
-				)
+					(reference "C8")
+					(unit 1)
+				)
