File: hardware/3axis-magnitometer/power.kicad_sch (KiCad schematic)
At the start: 16 parts, among them U3 AMS1117-3.3, U4 AMS1117-3.3

Commit message: Add files via upload
Parts:
- renumbered C13 to C15, C14 to C16, C15 to C17, C16 to C18, C17 to C20, C18 to C21, C19 to C22, C20 to C23, C21 to C24, C22 to C25, C23 to C26, C24 to C27, R13 to R12, R14 to R13, U3 to U5, U4 to U6
Changed lines of the file:
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@@
 		(dnp no)
 		(fields_autoplaced yes)
-		(property "Reference" "C14"
+		(property "Reference" "C16"
 			(at 148.59 104.1399 0)
 			(effects
@@
 			(project "3axis-magnitometer"
 				(path "/c590c88d-27c9-4e5a-a435-a42d9de70c1c/aa85cf22-72ca-4fb8-a4da-aecf61471964"
-					(reference "C14")
+					(reference "C16")
 					(unit 1)
 				)
@@
 		(dnp no)
 		(fields_autoplaced yes)
-		(property "Reference" "C13"
+		(property "Reference" "C15"
 			(at 148.59 85.0899 0)
 			(effects
@@
 			(project "3axis-magnitometer"
 				(path "/c590c88d-27c9-4e5a-a435-a42d9de70c1c/aa85cf22-72ca-4fb8-a4da-aecf61471964"
-					(reference "C13")
+					(reference "C15")
 					(unit 1)
 				)
@@
 		(dnp no)
 		(fields_autoplaced yes)
-		(property "Reference" "C21"
+		(property "Reference" "C24"
 			(at 212.09 104.1399 0)
 			(effects
@@
 			(project "3axis-magnitometer"
 				(path "/c590c88d-27c9-4e5a-a435-a42d9de70c1c/aa85cf22-72ca-4fb8-a4da-aecf61471964"
-					(reference "C21")
+					(reference "C24")
 					(unit 1)
 				)
@@
 		(dnp no)
 		(fields_autoplaced yes)
-		(property "Reference" "C24"
+		(property "Reference" "C27"
 			(at 226.06 85.0899 0)
 			(effects
@@
 			(project "3axis-magnitometer"
 				(path "/c590c88d-27c9-4e5a-a435-a42d9de70c1c/aa85cf22-72ca-4fb8-a4da-aecf61471964"
-					(reference "C24")
+					(reference "C27")
 					(unit 1)
 				)
@@
 		(dnp no)
 		(fields_autoplaced yes)
-		(property "Reference" "C22"
+		(property "Reference" "C25"
 			(at 215.9 85.0899 0)
 			(effects
@@
 			(project "3axis-magnitometer"
 				(path "/c590c88d-27c9-4e5a-a435-a42d9de70c1c/aa85cf22-72ca-4fb8-a4da-aecf61471964"
-					(reference "C22")
+					(reference "C25")
 					(unit 1)
 				)
@@
 		(on_board yes)
 		(dnp no)
-		(property "Reference" "R13"
+		(property "Reference" "R12"
 			(at 129.54 71.374 90)
 			(effects
@@
 			(project "3axis-magnitometer"
 				(path "/c590c88d-27c9-4e5a-a435-a42d9de70c1c/aa85cf22-72ca-4fb8-a4da-aecf61471964"
-					(reference "R13")
+					(reference "R12")
 					(unit 1)
 				)
@@
 		(dnp no)
 		(fields_autoplaced yes)
-		(property "Reference" "C15"
+		(property "Reference" "C17"
 			(at 158.75 85.0899 0)
 			(effects
@@
 			(project "3axis-magnitometer"
 				(path "/c590c88d-27c9-4e5a-a435-a42d9de70c1c/aa85cf22-72ca-4fb8-a4da-aecf61471964"
-					(reference "C15")
+					(reference "C17")
 					(unit 1)
 				)
@@
 		(dnp no)
 		(fields_autoplaced yes)
-		(property "Reference" "U4"
+		(property "Reference" "U6"
 			(at 180.34 92.71 0)
 			(effects
@@
 			(project "3axis-magnitometer"
 				(path "/c590c88d-27c9-4e5a-a435-a42d9de70c1c/aa85cf22-72ca-4fb8-a4da-aecf61471964"
-					(reference "U4")
+					(reference "U6")
 					(unit 1)
 				)
@@
 		(dnp no)
 		(fields_autoplaced yes)
-		(property "Reference" "C23"
+		(property "Reference" "C26"
 			(at 222.25 104.1399 0)
 			(effects
@@
 			(project "3axis-magnitometer"
 				(path "/c590c88d-27c9-4e5a-a435-a42d9de70c1c/aa85cf22-72ca-4fb8-a4da-aecf61471964"
-					(reference "C23")
+					(reference "C26")
 					(unit 1)
 				)
@@
 		(dnp no)
 		(fields_autoplaced yes)
-		(property "Reference" "C19"
+		(property "Reference" "C22"
 			(at 201.93 104.1399 0)
 			(effects
@@
 			(project ""
 				(path "/c590c88d-27c9-4e5a-a435-a42d9de70c1c/aa85cf22-72ca-4fb8-a4da-aecf61471964"
-					(reference "C19")
+					(reference "C22")
 					(unit 1)
 				)
@@
 		(dnp no)
 		(fields_autoplaced yes)
-		(property "Reference" "C16"
+		(property "Reference" "C18"
 			(at 158.75 104.1399 0)
 			(effects
@@
 			(project "3axis-magnitometer"
 				(path "/c590c88d-27c9-4e5a-a435-a42d9de70c1c/aa85cf22-72ca-4fb8-a4da-aecf61471964"
-					(reference "C16")
+					(reference "C18")
 					(unit 1)
 				)
@@
 		(on_board yes)
 		(dnp no)
-		(property "Reference" "R14"
+		(property "Reference" "R13"
 			(at 129.54 94.234 90)
 			(effects
@@
 			(project "3axis-magnitometer"
 				(path "/c590c88d-27c9-4e5a-a435-a42d9de70c1c/aa85cf22-72ca-4fb8-a4da-aecf61471964"
-					(reference "R14")
+					(reference "R13")
 					(unit 1)
 				)
@@
 		(dnp no)
 		(fields_autoplaced yes)
-		(property "Reference" "C17"
+		(property "Reference" "C20"
 			(at 168.91 85.0899 0)
 			(effects
@@
 			(project "3axis-magnitometer"
 				(path "/c590c88d-27c9-4e5a-a435-a42d9de70c1c/aa85cf22-72ca-4fb8-a4da-aecf61471964"
-					(reference "C17")
+					(reference "C20")
 					(unit 1)
 				)
@@
 		(dnp no)
 		(fields_autoplaced yes)
-		(property "Reference" "U3"
+		(property "Reference" "U5"
 			(at 180.34 69.85 0)
 			(effects
@@
 			(project ""
 				(path "/c590c88d-27c9-4e5a-a435-a42d9de70c1c/aa85cf22-72ca-4fb8-a4da-aecf61471964"
-					(reference "U3")
+					(reference "U5")
 					(unit 1)
 				)
@@
 		(dnp no)
 		(fields_autoplaced yes)
-		(property "Reference" "C20"
+		(property "Reference" "C23"
 			(at 205.74 85.0899 0)
 			(effects
@@
 			(project "3axis-magnitometer"
 				(path "/c590c88d-27c9-4e5a-a435-a42d9de70c1c/aa85cf22-72ca-4fb8-a4da-aecf61471964"
-					(reference "C20")
+					(reference "C23")
 					(unit 1)
 				)
@@
 		(dnp no)
 		(fields_autoplaced yes)
-		(property "Reference" "C18"
+		(property "Reference" "C21"
 			(at 168.91 104.1399 0)
 			(effects
@@
 			(project "3axis-magnitometer"
 				(path "/c590c88d-27c9-4e5a-a435-a42d9de70c1c/aa85cf22-72ca-4fb8-a4da-aecf61471964"
-					(reference "C18")
-					(unit 1)
-				)
+					(reference "C21")
+					(unit 1)
+				)

Commit message: начата новая трассировка
Parts:
- renumbered C15 to C16, C16 to C17, C17 to C18, C18 to C19, C20 to C21, C21 to C22, C22 to C23, C23 to C24, C24 to C25, C25 to C26, C26 to C27, C27 to C28
Changed lines of the file:
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@@
 		(dnp no)
 		(fields_autoplaced yes)
-		(property "Reference" "C16"
+		(property "Reference" "C17"
 			(at 148.59 104.1399 0)
 			(effects
@@
 			(project "3axis-magnitometer"
 				(path "/c590c88d-27c9-4e5a-a435-a42d9de70c1c/aa85cf22-72ca-4fb8-a4da-aecf61471964"
-					(reference "C16")
+					(reference "C17")
 					(unit 1)
 				)
@@
 		(dnp no)
 		(fields_autoplaced yes)
-		(property "Reference" "C15"
+		(property "Reference" "C16"
 			(at 148.59 85.0899 0)
 			(effects
@@
 			(project "3axis-magnitometer"
 				(path "/c590c88d-27c9-4e5a-a435-a42d9de70c1c/aa85cf22-72ca-4fb8-a4da-aecf61471964"
-					(reference "C15")
+					(reference "C16")
 					(unit 1)
 				)
@@
 		(dnp no)
 		(fields_autoplaced yes)
-		(property "Reference" "C24"
+		(property "Reference" "C25"
 			(at 212.09 104.1399 0)
 			(effects
@@
 			(project "3axis-magnitometer"
 				(path "/c590c88d-27c9-4e5a-a435-a42d9de70c1c/aa85cf22-72ca-4fb8-a4da-aecf61471964"
-					(reference "C24")
+					(reference "C25")
 					(unit 1)
 				)
@@
 		(dnp no)
 		(fields_autoplaced yes)
-		(property "Reference" "C27"
+		(property "Reference" "C28"
 			(at 226.06 85.0899 0)
 			(effects
@@
 			(project "3axis-magnitometer"
 				(path "/c590c88d-27c9-4e5a-a435-a42d9de70c1c/aa85cf22-72ca-4fb8-a4da-aecf61471964"
-					(reference "C27")
+					(reference "C28")
 					(unit 1)
 				)
@@
 		(dnp no)
 		(fields_autoplaced yes)
-		(property "Reference" "C25"
+		(property "Reference" "C26"
 			(at 215.9 85.0899 0)
 			(effects
@@
 			(project "3axis-magnitometer"
 				(path "/c590c88d-27c9-4e5a-a435-a42d9de70c1c/aa85cf22-72ca-4fb8-a4da-aecf61471964"
-					(reference "C25")
+					(reference "C26")
 					(unit 1)
 				)
@@
 		(dnp no)
 		(fields_autoplaced yes)
-		(property "Reference" "C17"
+		(property "Reference" "C18"
 			(at 158.75 85.0899 0)
 			(effects
@@
 			(project "3axis-magnitometer"
 				(path "/c590c88d-27c9-4e5a-a435-a42d9de70c1c/aa85cf22-72ca-4fb8-a4da-aecf61471964"
-					(reference "C17")
+					(reference "C18")
 					(unit 1)
 				)
@@
 		(dnp no)
 		(fields_autoplaced yes)
-		(property "Reference" "C26"
+		(property "Reference" "C27"
 			(at 222.25 104.1399 0)
 			(effects
@@
 			(project "3axis-magnitometer"
 				(path "/c590c88d-27c9-4e5a-a435-a42d9de70c1c/aa85cf22-72ca-4fb8-a4da-aecf61471964"
-					(reference "C26")
+					(reference "C27")
 					(unit 1)
 				)
@@
 		(dnp no)
 		(fields_autoplaced yes)
-		(property "Reference" "C22"
+		(property "Reference" "C23"
 			(at 201.93 104.1399 0)
 			(effects
@@
 			(project ""
 				(path "/c590c88d-27c9-4e5a-a435-a42d9de70c1c/aa85cf22-72ca-4fb8-a4da-aecf61471964"
-					(reference "C22")
+					(reference "C23")
 					(unit 1)
 				)
@@
 		(dnp no)
 		(fields_autoplaced yes)
-		(property "Reference" "C18"
+		(property "Reference" "C19"
 			(at 158.75 104.1399 0)
 			(effects
@@
 			(project "3axis-magnitometer"
 				(path "/c590c88d-27c9-4e5a-a435-a42d9de70c1c/aa85cf22-72ca-4fb8-a4da-aecf61471964"
-					(reference "C18")
+					(reference "C19")
 					(unit 1)
 				)
@@
 		(dnp no)
 		(fields_autoplaced yes)
-		(property "Reference" "C20"
+		(property "Reference" "C21"
 			(at 168.91 85.0899 0)
 			(effects
@@
 			(project "3axis-magnitometer"
 				(path "/c590c88d-27c9-4e5a-a435-a42d9de70c1c/aa85cf22-72ca-4fb8-a4da-aecf61471964"
-					(reference "C20")
+					(reference "C21")
 					(unit 1)
 				)
@@
 		(dnp no)
 		(fields_autoplaced yes)
-		(property "Reference" "C23"
+		(property "Reference" "C24"
 			(at 205.74 85.0899 0)
 			(effects
@@
 			(project "3axis-magnitometer"
 				(path "/c590c88d-27c9-4e5a-a435-a42d9de70c1c/aa85cf22-72ca-4fb8-a4da-aecf61471964"
-					(reference "C23")
+					(reference "C24")
 					(unit 1)
 				)
@@
 		(dnp no)
 		(fields_autoplaced yes)
-		(property "Reference" "C21"
+		(property "Reference" "C22"
 			(at 168.91 104.1399 0)
 			(effects
@@
 			(project "3axis-magnitometer"
 				(path "/c590c88d-27c9-4e5a-a435-a42d9de70c1c/aa85cf22-72ca-4fb8-a4da-aecf61471964"
-					(reference "C21")
-					(unit 1)
-				)
+					(reference "C22")
+					(unit 1)
+				)

Commit message: Финальные правки трассировки
Parts:
- renumbered C16 to C17, C17 to C18, C18 to C19, C19 to C20, C21 to C22, C22 to C23, C23 to C24, C24 to C25, C25 to C26, C26 to C27, C27 to C28, C28 to C29
Changed lines of the file:
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@@
 		(dnp no)
 		(fields_autoplaced yes)
-		(property "Reference" "C17"
+		(property "Reference" "C18"
 			(at 148.59 104.1399 0)
 			(effects
@@
 			(project "3axis-magnitometer"
 				(path "/c590c88d-27c9-4e5a-a435-a42d9de70c1c/aa85cf22-72ca-4fb8-a4da-aecf61471964"
-					(reference "C17")
+					(reference "C18")
 					(unit 1)
 				)
@@
 		(dnp no)
 		(fields_autoplaced yes)
-		(property "Reference" "C16"
+		(property "Reference" "C17"
 			(at 148.59 85.0899 0)
 			(effects
@@
 			(project "3axis-magnitometer"
 				(path "/c590c88d-27c9-4e5a-a435-a42d9de70c1c/aa85cf22-72ca-4fb8-a4da-aecf61471964"
-					(reference "C16")
+					(reference "C17")
 					(unit 1)
 				)
@@
 		(dnp no)
 		(fields_autoplaced yes)
-		(property "Reference" "C25"
+		(property "Reference" "C26"
 			(at 212.09 104.1399 0)
 			(effects
@@
 			(project "3axis-magnitometer"
 				(path "/c590c88d-27c9-4e5a-a435-a42d9de70c1c/aa85cf22-72ca-4fb8-a4da-aecf61471964"
-					(reference "C25")
+					(reference "C26")
 					(unit 1)
 				)
@@
 		(dnp no)
 		(fields_autoplaced yes)
-		(property "Reference" "C28"
+		(property "Reference" "C29"
 			(at 226.06 85.0899 0)
 			(effects
@@
 			(project "3axis-magnitometer"
 				(path "/c590c88d-27c9-4e5a-a435-a42d9de70c1c/aa85cf22-72ca-4fb8-a4da-aecf61471964"
-					(reference "C28")
+					(reference "C29")
 					(unit 1)
 				)
@@
 		(dnp no)
 		(fields_autoplaced yes)
-		(property "Reference" "C26"
+		(property "Reference" "C27"
 			(at 215.9 85.0899 0)
 			(effects
@@
 			(project "3axis-magnitometer"
 				(path "/c590c88d-27c9-4e5a-a435-a42d9de70c1c/aa85cf22-72ca-4fb8-a4da-aecf61471964"
-					(reference "C26")
+					(reference "C27")
 					(unit 1)
 				)
@@
 		(dnp no)
 		(fields_autoplaced yes)
-		(property "Reference" "C18"
+		(property "Reference" "C19"
 			(at 158.75 85.0899 0)
 			(effects
@@
 			(project "3axis-magnitometer"
 				(path "/c590c88d-27c9-4e5a-a435-a42d9de70c1c/aa85cf22-72ca-4fb8-a4da-aecf61471964"
-					(reference "C18")
+					(reference "C19")
 					(unit 1)
 				)
@@
 		(dnp no)
 		(fields_autoplaced yes)
-		(property "Reference" "C27"
+		(property "Reference" "C28"
 			(at 222.25 104.1399 0)
 			(effects
@@
 			(project "3axis-magnitometer"
 				(path "/c590c88d-27c9-4e5a-a435-a42d9de70c1c/aa85cf22-72ca-4fb8-a4da-aecf61471964"
-					(reference "C27")
+					(reference "C28")
 					(unit 1)
 				)
@@
 		(dnp no)
 		(fields_autoplaced yes)
-		(property "Reference" "C23"
+		(property "Reference" "C24"
 			(at 201.93 104.1399 0)
 			(effects
@@
 			(project ""
 				(path "/c590c88d-27c9-4e5a-a435-a42d9de70c1c/aa85cf22-72ca-4fb8-a4da-aecf61471964"
-					(reference "C23")
+					(reference "C24")
 					(unit 1)
 				)
@@
 		(dnp no)
 		(fields_autoplaced yes)
-		(property "Reference" "C19"
+		(property "Reference" "C20"
 			(at 158.75 104.1399 0)
 			(effects
@@
 			(project "3axis-magnitometer"
 				(path "/c590c88d-27c9-4e5a-a435-a42d9de70c1c/aa85cf22-72ca-4fb8-a4da-aecf61471964"
-					(reference "C19")
+					(reference "C20")
 					(unit 1)
 				)
@@
 		(dnp no)
 		(fields_autoplaced yes)
-		(property "Reference" "C21"
+		(property "Reference" "C22"
 			(at 168.91 85.0899 0)
 			(effects
@@
 			(project "3axis-magnitometer"
 				(path "/c590c88d-27c9-4e5a-a435-a42d9de70c1c/aa85cf22-72ca-4fb8-a4da-aecf61471964"
-					(reference "C21")
+					(reference "C22")
 					(unit 1)
 				)
@@
 		(dnp no)
 		(fields_autoplaced yes)
-		(property "Reference" "C24"
+		(property "Reference" "C25"
 			(at 205.74 85.0899 0)
 			(effects
@@
 			(project "3axis-magnitometer"
 				(path "/c590c88d-27c9-4e5a-a435-a42d9de70c1c/aa85cf22-72ca-4fb8-a4da-aecf61471964"
-					(reference "C24")
+					(reference "C25")
 					(unit 1)
 				)
@@
 		(dnp no)
 		(fields_autoplaced yes)
-		(property "Reference" "C22"
+		(property "Reference" "C23"
 			(at 168.91 104.1399 0)
 			(effects
@@
 			(project "3axis-magnitometer"
 				(path "/c590c88d-27c9-4e5a-a435-a42d9de70c1c/aa85cf22-72ca-4fb8-a4da-aecf61471964"
-					(reference "C22")
-					(unit 1)
-				)
+					(reference "C23")
+					(unit 1)
+				)
