File: hardware/3axis-magnitometer/sd-card.kicad_sch (KiCad schematic)
At the start: 4 parts, among them J2 Micro_SD_Card

Commit message: Add files via upload
Parts:
- removed J2: Micro_SD_Card, Connector_Card:microSD_HC_Molex_47219-2001, symbol Connector:Micro_SD_Card
- added U2: W25Q128JVS, Package_SO:SOIC-8_5.3x5.3mm_P1.27mm, symbol Memory_Flash:W25Q128JVS
- renumbered C5 to C4, C4 to C5, R5 to R2
Connections:
- net CLK: now also U2.6 (CLK)
- net CS: now also U2.1 (~{CS})
- net GND: now also U2.4 (GND)
- net MISO: now also U2.2 (DO/IO_{1})
- net MOSI: now also U2.5 (DI/IO_{0})
- net at C4.2, C5.2, R2.2: now also U2.3 (~{WP}/IO_{2}), U2.7 (~{HOLD}/~{RESET}/IO_{3}), U2.8 (VCC)
- no-connect marks 2 -> 0
Other:
- moved on the sheet: C4, C5, R2

Commit message: начата новая трассировка
Parts:
- renumbered C4 to C5, C5 to C6
Changed lines of the file:
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@@
 		(on_board yes)
 		(dnp no)
-		(property "Reference" "C5"
+		(property "Reference" "C6"
 			(at 229.87 71.374 0)
 			(effects
@@
 			(project ""
 				(path "/c590c88d-27c9-4e5a-a435-a42d9de70c1c/a46e14a1-6a3b-4c39-b96c-ca31b85d9e43"
-					(reference "C5")
+					(reference "C6")
 					(unit 1)
 				)
@@
 		(on_board yes)
 		(dnp no)
-		(property "Reference" "C4"
+		(property "Reference" "C5"
 			(at 214.9078 70.8881 0)
 			(effects
@@
 			(project "3axis-magnitometer"
 				(path "/c590c88d-27c9-4e5a-a435-a42d9de70c1c/a46e14a1-6a3b-4c39-b96c-ca31b85d9e43"
-					(reference "C4")
-					(unit 1)
-				)
+					(reference "C5")
+					(unit 1)
+				)

Commit message: трасировка магнитометра
Parts:
- U2: footprint Package_SO:SOIC-8_5.3x5.3mm_P1.27mm -> Package_SO:SOIC-8_3.9x4.9mm_P1.27mm
Changed lines of the file:
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@@
 			)
 		)
-		(property "Footprint" "Package_SO:SOIC-8_5.3x5.3mm_P1.27mm"
+		(property "Footprint" "Package_SO:SOIC-8_3.9x4.9mm_P1.27mm"
 			(at 181.61 45.72 0)
 			(effects

Commit message: Финальные правки трассировки
Parts:
- renumbered C5 to C6, C6 to C7
Changed lines of the file:
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@@
 		(on_board yes)
 		(dnp no)
-		(property "Reference" "C6"
+		(property "Reference" "C7"
 			(at 229.87 71.374 0)
 			(effects
@@
 			(project ""
 				(path "/c590c88d-27c9-4e5a-a435-a42d9de70c1c/a46e14a1-6a3b-4c39-b96c-ca31b85d9e43"
-					(reference "C6")
+					(reference "C7")
 					(unit 1)
 				)
@@
 		(on_board yes)
 		(dnp no)
-		(property "Reference" "C5"
+		(property "Reference" "C6"
 			(at 214.9078 70.8881 0)
 			(effects
@@
 			(project "3axis-magnitometer"
 				(path "/c590c88d-27c9-4e5a-a435-a42d9de70c1c/a46e14a1-6a3b-4c39-b96c-ca31b85d9e43"
-					(reference "C5")
-					(unit 1)
-				)
+					(reference "C6")
+					(unit 1)
+				)
